File: Electrical/ferrofluid_display/ferrofluid_display.kicad_pcb (KiCad board)
At the start: 2 copper layers, 627 parts, among them J1001 Screw_Terminal_01x06, U100001 DRV8872DDAR, U10001 DRV8872DDAR, U1001 74HC595, U101001 DRV8872DDAR, U102001 DRV8872DDAR, U103001 DRV8872DDAR, U105001 DRV8872DDAR, U106001 DRV8872DDAR, U107001 DRV8872DDAR, U108001 DRV8872DDAR, U109001 DRV8872DDAR, U110001 DRV8872DDAR, U11001 DRV8872DDAR, U111001 DRV8872DDAR, U112001 DRV8872DDAR, U113001 DRV8872DDAR, U114001 DRV8872DDAR, U12001 DRV8872DDAR, U13001 DRV8872DDAR, U14001 DRV8872DDAR, U15001 DRV8872DDAR, U17001 DRV8872DDAR, U18001 DRV8872DDAR, U19001 DRV8872DDAR, U20001 DRV8872DDAR, U2002 74HC595, U2003 74HC595, U2004 74HC595, U2005 74HC595, U2006 74HC595, U2007 74HC595, U2008 74HC595, U2009 74HC595, U21001 DRV8872DDAR, U22001 DRV8872DDAR, U23001 DRV8872DDAR, U24001 DRV8872DDAR, U25001 DRV8872DDAR, U26001 DRV8872DDAR, U28001 DRV8872DDAR, U29001 DRV8872DDAR, U30001 DRV8872DDAR, U3002 74HC595, U3003 74HC595, U3004 74HC595, U3005 74HC595, U3006 74HC595, U3007 74HC595, U3008 74HC595, U3009 74HC595, U31001 DRV8872DDAR, U32001 DRV8872DDAR, U33001 DRV8872DDAR, U34001 DRV8872DDAR, U35001 DRV8872DDAR, U36001 DRV8872DDAR, U37001 DRV8872DDAR, U39001 DRV8872DDAR, U40001 DRV8872DDAR, U4002 74HC595, U4003 74HC595, U4004 74HC595, U4005 74HC595, U4006 74HC595, U4007 74HC595, U4008 74HC595, U4009 74HC595, U41001 DRV8872DDAR, U42001 DRV8872DDAR, U43001 DRV8872DDAR, U44001 DRV8872DDAR, U45001 DRV8872DDAR, U46001 DRV8872DDAR, U47001 DRV8872DDAR, U48001 DRV8872DDAR, U50001 DRV8872DDAR, U51001 DRV8872DDAR, U52001 DRV8872DDAR, U53001 DRV8872DDAR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

Commit message: Started scripting
Parts:
- moved R77002 18.9 mm to (132.2, 7.25)
- moved D77001 18.4 mm to (133.0, 9.25)
- moved R77001 9.56 mm to (136.5, 9.25)
- moved D77002 9.04 mm to (135.8, 7.25), turned to 180 degrees
- moved L77001 7.67 mm to (140.0, 12.2), turned to 90 degrees
Changed lines of the file:
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@@
-(kicad_pcb (version 20171130) (host pcbnew "(5.0.0-rc2-dev-668-g07e7340a9)")
+(kicad_pcb (version 4) (host pcbnew 4.0.4-snap1-stable)
   (general
+    (links 1588)
+    (no_connects 1588)
+    (area -9 1.4825 381.348333 227.2525)
     (thickness 1.6)
     (drawings 0)
@@
     (46 B.CrtYd user)
     (47 F.CrtYd user)
-    (48 B.Fab user)
-    (49 F.Fab user)
+    (48 B.Fab user hide)
+    (49 F.Fab user hide)
   )
   (setup
@@
       (layerselection 0x010fc_ffffffff)
       (usegerberextensions false)
-      (usegerberattributes false)
-      (usegerberadvancedattributes false)
-      (creategerberjobfile false)
       (excludeedgelayer true)
       (linewidth 0.100000)
@@
       (hpglpenspeed 20)
       (hpglpendiameter 15)
+      (hpglpenoverlay 2)
       (psnegative false)
       (psa4output false)
@@
   )
   (module LEDs:LED_0805 (layer F.Cu)
-    (at 150.631666 3.9075)
+    (at 133 9.25)
     (descr "LED 0805 smd package")
     (tags "LED led 0805 SMD smd SMT smt smdled SMDLED smtled SMTLED")
     (attr smd)
-    (fp_text reference D77001 (at 0 -1.45) (layer F.SilkS)
-      (effects (font (size 1 1) (thickness 0.15)))
+    (fp_text reference D77001 (at -2.75 0 90) (layer F.SilkS)
+      (effects (font (size 0.5 0.5) (thickness 0.1)))
     )
     (fp_text value GREEN_LED (at 0 1.55) (layer F.Fab)
@@
   )
   (module LEDs:LED_0805 (layer F.Cu)
-    (at 143.994047 10.9575)
+    (at 135.75 7.25 180)
     (descr "LED 0805 smd package")
     (tags "LED led 0805 SMD smd SMT smt smdled SMDLED smtled SMTLED")
     (attr smd)
-    (fp_text reference D77002 (at 0 -1.45) (layer F.SilkS)
-      (effects (font (size 1 1) (thickness 0.15)))
+    (fp_text reference D77002 (at -3.5 0 180) (layer F.SilkS)
+      (effects (font (size 0.5 0.5) (thickness 0.1)))
     )
-    (fp_text value BLUE_LED (at 0 1.55) (layer F.Fab)
+    (fp_text value BLUE_LED (at 0 1.55 180) (layer F.Fab)
       (effects (font (size 1 1) (thickness 0.15)))
     )
-    (fp_text user %R (at 0 -1.25) (layer F.Fab)
+    (fp_text user %R (at 0 -1.25 180) (layer F.Fab)
       (effects (font (size 0.4 0.4) (thickness 0.1)))
     )
@@
     (fp_line (start -0.4 -0.4) (end -0.4 0.4) (layer F.Fab) (width 0.1))
     (fp_line (start -1.8 -0.7) (end -1.8 0.7) (layer F.SilkS) (width 0.12))
-    (pad 1 smd rect (at -1.1 0 180) (size 1.2 1.2) (layers F.Cu F.Paste F.Mask)
+    (pad 1 smd rect (at -1.1 0) (size 1.2 1.2) (layers F.Cu F.Paste F.Mask)
       (net 291 "Net-(D77002-Pad1)"))
-    (pad 2 smd rect (at 1.1 0 180) (size 1.2 1.2) (layers F.Cu F.Paste F.Mask)
+    (pad 2 smd rect (at 1.1 0) (size 1.2 1.2) (layers F.Cu F.Paste F.Mask)
       (net 292 "Net-(D77002-Pad2)"))
     (model ${KISYS3DMOD}/LEDs.3dshapes/LED_0805.wrl
@@
   )
   (module CustomFootprints:ElectroMagnet (layer F.Cu)
-    (at 137.614524 4.9575)
-    (fp_text reference L77001 (at 0 2.5) (layer F.SilkS)
-      (effects (font (size 1 1) (thickness 0.15)))
+    (at 140 12.25 90)
+    (fp_text reference L77001 (at 0 2 90) (layer F.SilkS)
+      (effects (font (size 0.5 0.5) (thickness 0.1)))
     )
-    (fp_text value Electromagnetic_Actor (at 0 -2.5) (layer F.Fab)
+    (fp_text value Electromagnetic_Actor (at 0 -2.5 90) (layer F.Fab)
       (effects (font (size 1 1) (thickness 0.15)))
     )
@@
     (fp_line (start -2.5 1.5) (end 2.5 1.5) (layer F.SilkS) (width 0.15))
     (fp_line (start -2.5 -1.5) (end -2.5 1.5) (layer F.SilkS) (width 0.15))
-    (pad 2 thru_hole circle (at 1.5 0) (size 1.524 1.524) (drill 0.762) (layers *.Cu *.Mask)
+    (pad 2 thru_hole circle (at 1.5 0 90) (size 1.524 1.524) (drill 0.762) (layers *.Cu *.Mask)
       (net 290 "Net-(D77001-Pad1)"))
-    (pad 1 thru_hole circle (at -1.5 0) (size 1.524 1.524) (drill 0.762) (layers *.Cu *.Mask)
+    (pad 1 thru_hole circle (at -1.5 0 90) (size 1.524 1.524) (drill 0.762) (layers *.Cu *.Mask)
       (net 291 "Net-(D77002-Pad1)"))
   )
@@
   )
   (module Resistors_SMD:R_0603 (layer F.Cu)
-    (at 143.255952 16.0075)
+    (at 136.5 9.25)
     (descr "Resistor SMD 0603, reflow soldering, Vishay (see dcrcw.pdf)")
     (tags "resistor 0603")
     (attr smd)
-    (fp_text reference R77001 (at 0 -1.45) (layer F.SilkS)
-      (effects (font (size 1 1) (thickness 0.15)))
+    (fp_text reference R77001 (at 2.75 0 180) (layer F.SilkS)
+      (effects (font (size 0.5 0.5) (thickness 0.1)))
     )
     (fp_text value 1k (at 0 1.5) (layer F.Fab)
@@
   )
   (module Resistors_SMD:R_0603 (layer F.Cu)
-    (at 151.035952 8.9575)
+    (at 132.25 7.25)
     (descr "Resistor SMD 0603, reflow soldering, Vishay (see dcrcw.pdf)")
     (tags "resistor 0603")
     (attr smd)
-    (fp_text reference R77002 (at 0 -1.45) (layer F.SilkS)
-      (effects (font (size 1 1) (thickness 0.15)))
+    (fp_text reference R77002 (at 0 -1.25) (layer F.SilkS)
+      (effects (font (size 0.5 0.5) (thickness 0.1)))
     )
     (fp_text value 1k (at 0 1.5) (layer F.Fab)
@@
     (tags "HTSOP 1.27")
     (attr smd)
-    (fp_text reference U77001 (at 0 -3.5) (layer F.SilkS)
-      (effects (font (size 1 1) (thickness 0.15)))
+    (fp_text reference U77001 (at -4.316905 -0.0075 90) (layer F.SilkS)
+      (effects (font (size 0.5 0.5) (thickness 0.1)))
     )
     (fp_text value DRV8872DDAR (at 0 3.5) (layer F.Fab)
