File: Electrical/ferrofluid_display/ferrofluid_display_original.kicad_pcb (KiCad board)
At the start: 2 copper layers, 627 parts, among them J1001 Screw_Terminal_01x06, U100001 DRV8872DDAR, U10001 DRV8872DDAR, U1001 74HC595, U101001 DRV8872DDAR, U102001 DRV8872DDAR, U103001 DRV8872DDAR, U105001 DRV8872DDAR, U106001 DRV8872DDAR, U107001 DRV8872DDAR, U108001 DRV8872DDAR, U109001 DRV8872DDAR, U110001 DRV8872DDAR, U11001 DRV8872DDAR, U111001 DRV8872DDAR, U112001 DRV8872DDAR, U113001 DRV8872DDAR, U114001 DRV8872DDAR, U12001 DRV8872DDAR, U13001 DRV8872DDAR, U14001 DRV8872DDAR, U15001 DRV8872DDAR, U17001 DRV8872DDAR, U18001 DRV8872DDAR, U19001 DRV8872DDAR, U20001 DRV8872DDAR, U2002 74HC595, U2003 74HC595, U2004 74HC595, U2005 74HC595, U2006 74HC595, U2007 74HC595, U2008 74HC595, U2009 74HC595, U21001 DRV8872DDAR, U22001 DRV8872DDAR, U23001 DRV8872DDAR, U24001 DRV8872DDAR, U25001 DRV8872DDAR, U26001 DRV8872DDAR, U28001 DRV8872DDAR, U29001 DRV8872DDAR, U30001 DRV8872DDAR, U3002 74HC595, U3003 74HC595, U3004 74HC595, U3005 74HC595, U3006 74HC595, U3007 74HC595, U3008 74HC595, U3009 74HC595, U31001 DRV8872DDAR, U32001 DRV8872DDAR, U33001 DRV8872DDAR, U34001 DRV8872DDAR, U35001 DRV8872DDAR, U36001 DRV8872DDAR, U37001 DRV8872DDAR, U39001 DRV8872DDAR, U40001 DRV8872DDAR, U4002 74HC595, U4003 74HC595, U4004 74HC595, U4005 74HC595, U4006 74HC595, U4007 74HC595, U4008 74HC595, U4009 74HC595, U41001 DRV8872DDAR, U42001 DRV8872DDAR, U43001 DRV8872DDAR, U44001 DRV8872DDAR, U45001 DRV8872DDAR, U46001 DRV8872DDAR, U47001 DRV8872DDAR, U48001 DRV8872DDAR, U50001 DRV8872DDAR, U51001 DRV8872DDAR, U52001 DRV8872DDAR, U53001 DRV8872DDAR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

Commit message: Auto-layed out file
Routing:
- net GND: track 0.00 -> 3.41 mm, vias 0 -> 2
Changed lines of the file:
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@@
     (thickness 1.6)
     (drawings 0)
-    (tracks 22)
+    (tracks 28)
     (zones 0)
     (modules 627)
@@
   )
   (setup
-    (last_trace_width 0.25)
+    (last_trace_width 0.5)
     (user_trace_width 0.5)
     (trace_clearance 0.2)
@@
     )
   )
+  (via (at 139.7 -8.382) (size 0.8) (drill 0.4) (layers F.Cu B.Cu) (net 5))
+  (segment (start 139.4945 -8.5875) (end 139.7 -8.382) (width 0.5) (layer F.Cu) (net 5))
+  (segment (start 138.156905 -8.5875) (end 139.4945 -8.5875) (width 0.5) (layer F.Cu) (net 5))
+  (via (at 131.064 -9.652) (size 0.8) (drill 0.4) (layers F.Cu B.Cu) (net 5))
+  (segment (start 131.2695 -9.8575) (end 131.064 -9.652) (width 0.5) (layer F.Cu) (net 5))
+  (segment (start 132.756905 -9.8575) (end 131.2695 -9.8575) (width 0.5) (layer F.Cu) (net 5))
   (segment (start 138.386405 -9.628) (end 138.156905 -9.8575) (width 0.5) (layer F.Cu) (net 29))
   (segment (start 141.224 -9.628) (end 138.386405 -9.628) (width 0.5) (layer F.Cu) (net 29))
@@
     (polygon
       (pts
-        (xy 131.064 -15.748) (xy 131.064 -4.064) (xy 143.256 -4.064) (xy 143.256 -15.748)
+        (xy 130.556 -15.748) (xy 130.556 -4.064) (xy 143.256 -4.064) (xy 143.256 -15.748)
       )
     )
