File: Electrical/ferrofluid_display/ferrofluid_display.sch (KiCad schematic (older format))
At the start: 4 parts

Commit message: Schematic complete, layout starting
Parts:
- removed Q? (x2): PDFN33, symbol Custom:PDFN33
- removed Q?: CPH5504-TL-E, symbol Custom:CPH5504-TL-E
- added J1001: Screw_Terminal_01x06, CustomFootprints:399700106, symbol Connector:Screw_Terminal_01x06
- added U1001: 74HC595, CustomFootprints:74HC595D, symbol 74xx:74HC595
- A1001: renamed from A?; footprint (none) -> Modules:Arduino_Nano
Connections:
- net labels added: +12V, +3V3, +5V, GND, O_1, O_10, O_100, O_101, O_102, O_103, O_104, O_105, O_106, O_107, O_108, O_109, O_11, O_110, O_111, O_112, O_113, O_114, O_115, O_116, O_117, O_118, O_119, O_12, O_120, O_121, O_122, O_123, O_124, O_125, O_126, O_127, O_128, O_129, O_13, O_130, O_131, O_132, O_133, O_134, O_135, O_136, O_137, O_138, O_139, O_14, O_140, O_141, O_142, O_143, O_144, O_145, O_146, O_147, O_148, O_149, O_15, O_150, O_151, O_152, O_153, O_154, O_155, O_156, O_157, O_158, O_159, O_16, O_160, O_161, O_162, O_163, O_164, O_165, O_166, O_167, O_168, O_169, O_17, O_170, O_171, O_172, O_173, O_174, O_175, O_176, O_177, O_178, O_179, O_18, O_180, O_181, O_182, O_183, O_184, O_185, O_186, O_187, O_188, O_189, O_19, O_190, O_191, O_192, O_193, O_194, O_195, O_196, O_197, O_198, O_199, O_2, O_20, O_200, O_21, O_22, O_23, O_24, O_25, O_26, O_27, O_28, O_29, O_3, O_30, O_31, O_32, O_33, O_34, O_35, O_36, O_37, O_38, O_39, O_4, O_40, O_41, O_42, O_43, O_44, O_45, O_46, O_47, O_48, O_49, O_5, O_50, O_51, O_52, O_53, O_54, O_55, O_56, O_57, O_58, O_59, O_6, O_60, O_61, O_62, O_63, O_64, O_65, O_66, O_67, O_68, O_69, O_7, O_70, O_71, O_72, O_73, O_74, O_75, O_76, O_77, O_78, O_79, O_8, O_80, O_81, O_82, O_83, O_84, O_85, O_86, O_87, O_88, O_89, O_9, O_90, O_91, O_92, O_93, O_94, O_95, O_96, O_97, O_98, O_99, RCLK, SER, SER_1_2, SER_2_3, SER_3_F, SRCLK, SRCLR
- wire segments 0 -> 25
- no-connect marks 0 -> 21
Other:
- moved on the sheet: A1001

Commit message: Started scripting
Changed lines of the file:
@@
-EESchema Schematic File Version 4
+EESchema Schematic File Version 2
+LIBS:power
 LIBS:ferrofluid_display-cache
-EELAYER 26 0
+EELAYER 25 0
 EELAYER END
 $Descr A4 11693 8268
@@
 O_192
 $Comp
-L power:GND #PWR01001
+L power:GND #PWR01
 U 1 1 5BEA829C
 P 8225 2325
-F 0 "#PWR01001" H 8225 2075 50  0001 C CNN
+F 0 "#PWR01" H 8225 2075 50  0001 C CNN
 F 1 "GND" H 8230 2152 50  0000 C CNN
 F 2 "" H 8225 2325 50  0001 C CNN
@@
 O_200
 $Comp
-L power:+12V #PWR01002
+L power:+12V #PWR02
 U 1 1 5BF64A73
 P 8825 750
-F 0 "#PWR01002" H 8825 600 50  0001 C CNN
+F 0 "#PWR02" H 8825 600 50  0001 C CNN
 F 1 "+12V" H 8840 923 50  0000 C CNN
 F 2 "" H 8825 750 50  0001 C CNN
@@
 $EndComp
 $Comp
-L power:GND #PWR01003
+L power:GND #PWR03
 U 1 1 5BF64ABC
 P 8825 1450
-F 0 "#PWR01003" H 8825 1200 50  0001 C CNN
+F 0 "#PWR03" H 8825 1200 50  0001 C CNN
 F 1 "GND" H 8830 1277 50  0000 C CNN
 F 2 "" H 8825 1450 50  0001 C CNN
@@
 $EndComp
 Wire Wire Line
-	8825 1450 8825 1325
+	8825 1125 8825 1450
 Wire Wire Line
 	8825 1125 8900 1125
 Wire Wire Line
-	8900 1025 8825 1025
-Wire Wire Line
-	8825 1025 8825 925
+	8600 1025 8900 1025
+Wire Wire Line
+	8825 750  8825 1025
 Wire Wire Line
 	8900 1225 8825 1225
 Connection ~ 8825 1225
 Wire Wire Line
-	8825 1225 8825 1125
-Wire Wire Line
-	8900 925  8825 925
+	8825 925  8900 925
 Connection ~ 8825 925
-Wire Wire Line
-	8825 925  8825 825
 $Comp
 L Connector:Screw_Terminal_01x06 J1001
@@
 $EndComp
 Wire Wire Line
-	8900 1325 8825 1325
+	8825 1325 8900 1325
 Connection ~ 8825 1325
-Wire Wire Line
-	8825 1325 8825 1225
 Wire Wire Line
 	8900 825  8825 825
 Connection ~ 8825 825
-Wire Wire Line
-	8825 825  8825 750
 $Comp
-L power:+12V #PWR0101
+L power:+12V #PWR04
 U 1 1 5BF682F9
 P 6475 2250
-F 0 "#PWR0101" H 6475 2100 50  0001 C CNN
+F 0 "#PWR04" H 6475 2100 50  0001 C CNN
 F 1 "+12V" V 6490 2378 50  0000 L CNN
 F 2 "" H 6475 2250 50  0001 C CNN
@@
 	6575 2250 6575 2225
 $Comp
-L power:+5V #PWR0102
+L power:+5V #PWR05
 U 1 1 5BF6846A
 P 6675 2325
-F 0 "#PWR0102" H 6675 2175 50  0001 C CNN
+F 0 "#PWR05" H 6675 2175 50  0001 C CNN
 F 1 "+5V" V 6690 2453 50  0000 L CNN
 F 2 "" H 6675 2325 50  0001 C CNN
@@
 $EndComp
 Wire Wire Line
-	6675 2325 6675 2275
+	6675 2225 6675 2325
 $Comp
-L power:+3V3 #PWR0103
+L power:+3V3 #PWR06
 U 1 1 5BF68B47
 P 6775 2425
-F 0 "#PWR0103" H 6775 2275 50  0001 C CNN
+F 0 "#PWR06" H 6775 2275 50  0001 C CNN
 F 1 "+3V3" V 6790 2553 50  0000 L CNN
 F 2 "" H 6775 2425 50  0001 C CNN
@@
 $EndComp
 Wire Wire Line
-	6775 2425 6775 2375
+	6775 2225 6775 2425
 NoConn ~ 7875 875
 NoConn ~ 7975 875
@@
 NoConn ~ 7375 2225
 $Comp
-L power:PWR_FLAG #FLG0101
+L power:PWR_FLAG #FLG07
 U 1 1 5BF70B0C
 P 8600 1025
-F 0 "#FLG0101" H 8600 1100 50  0001 C CNN
+F 0 "#FLG07" H 8600 1100 50  0001 C CNN
 F 1 "PWR_FLAG" H 8600 1199 50  0000 C CNN
 F 2 "" H 8600 1025 50  0001 C CNN
@@
 	1    0    0    -1
 $EndComp
-Wire Wire Line
-	8825 1025 8600 1025
 Connection ~ 8825 1025
 $Comp
-L power:PWR_FLAG #FLG0102
+L power:PWR_FLAG #FLG08
 U 1 1 5BF7101F
 P 6775 2375
-F 0 "#FLG0102" H 6775 2450 50  0001 C CNN
+F 0 "#FLG08" H 6775 2450 50  0001 C CNN
 F 1 "PWR_FLAG" V 6775 2503 50  0000 L CNN
 F 2 "" H 6775 2375 50  0001 C CNN
@@
 $EndComp
 Connection ~ 6775 2375
-Wire Wire Line
-	6775 2375 6775 2225
 $Comp
-L power:PWR_FLAG #FLG0103
+L power:PWR_FLAG #FLG09
 U 1 1 5BF71049
 P 6675 2275
-F 0 "#FLG0103" H 6675 2350 50  0001 C CNN
+F 0 "#FLG09" H 6675 2350 50  0001 C CNN
 F 1 "PWR_FLAG" V 6675 2403 50  0000 L CNN
 F 2 "" H 6675 2275 50  0001 C CNN
@@
 $EndComp
 Connection ~ 6675 2275
-Wire Wire Line
-	6675 2275 6675 2225
 $Sheet
 S 1000 800  1050 6450
@@
 $EndComp
 $Comp
-L power:GND #PWR0104
+L power:GND #PWR010
 U 1 1 5C14E365
 P 9625 1575
-F 0 "#PWR0104" H 9625 1325 50  0001 C CNN
+F 0 "#PWR010" H 9625 1325 50  0001 C CNN
 F 1 "GND" H 9630 1402 50  0000 C CNN
 F 2 "" H 9625 1575 50  0001 C CNN
@@
 	9725 1575 9625 1575
 $Comp
-L power:GND #PWR0105
+L power:GND #PWR011
 U 1 1 5C14E36C
 P 10225 2225
-F 0 "#PWR0105" H 10225 1975 50  0001 C CNN
+F 0 "#PWR011" H 10225 1975 50  0001 C CNN
 F 1 "GND" H 10230 2052 50  0000 C CNN
 F 2 "" H 10225 2225 50  0001 C CNN
@@
 	10225 2175 10225 2225
 $Comp
-L power:+5V #PWR0106
+L power:+5V #PWR012
 U 1 1 5C14E376
 P 10225 625
-F 0 "#PWR0106" H 10225 475 50  0001 C CNN
+F 0 "#PWR012" H 10225 475 50  0001 C CNN
 F 1 "+5V" H 10240 798 50  0000 C CNN
 F 2 "" H 10225 625 50  0001 C CNN

Commit message: Added layers and 5V via
Changed lines of the file:
@@
-EESchema Schematic File Version 2
-LIBS:power
+EESchema Schematic File Version 4
 LIBS:ferrofluid_display-cache
-EELAYER 25 0
+EELAYER 26 0
 EELAYER END
 $Descr A4 11693 8268
@@
 $EndComp
 Wire Wire Line
-	8825 1125 8825 1450
+	8825 1125 8825 1225
 Wire Wire Line
 	8825 1125 8900 1125
 Wire Wire Line
-	8600 1025 8900 1025
-Wire Wire Line
-	8825 750  8825 1025
+	8600 1025 8825 1025
+Wire Wire Line
+	8825 750  8825 825
 Wire Wire Line
 	8900 1225 8825 1225
@@
 $EndComp
 Wire Wire Line
-	6675 2225 6675 2325
+	6675 2225 6675 2275
 $Comp
 L power:+3V3 #PWR06
@@
 $EndComp
 Wire Wire Line
-	6775 2225 6775 2425
+	6775 2225 6775 2375
 NoConn ~ 7875 875
 NoConn ~ 7975 875
@@
 NoConn ~ 7675 875
 NoConn ~ 7775 875
+Wire Wire Line
+	8825 1225 8825 1325
+Wire Wire Line
+	8825 925  8825 1025
+Wire Wire Line
+	8825 1325 8825 1450
+Wire Wire Line
+	8825 825  8825 925
+Wire Wire Line
+	8825 1025 8900 1025
+Wire Wire Line
+	6775 2375 6775 2425
+Wire Wire Line
+	6675 2275 6675 2325
 $EndSCHEMATC
